File: Buck/Buck.kicad_sch (KiCad schematic)
At the start: 7 parts, among them U2 APE1707S-50-HF

Commit message: Buck_Converter(12-24V)(3.3-5V)
Other:
- note added: "Daca am nevoie de Vin la o tensiune mai mare(V) am nevoie de un alt chip(U2)"
Changed lines of the file:
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@@
+		)
+	)
+	(text "Daca am nevoie de Vin la o tensiune mai mare(V) am nevoie de un alt chip(U2) "
+		(exclude_from_sim no)
+		(at 150.622 73.66 0)
+		(effects
+			(font
+				(size 1.27 1.27)
+			)
 		)
 	)

Commit message: 2.Better version
Parts:
- added R1, R2: R_Small, symbol Device:R_Small
Connections:
- net GND: now also R2.2
- net Vout: now also R1.1; no longer U2.4 (FB)
- new net: R1.2, R2.1, U2.4 (FB)
Other:
- moved on the sheet: C1, C2, C3, C4, D1, L1, U2

Commit message: 3.0
Other:
- note added: "https://pdf.datasheet.live/datasheets-1/advanced_power_electronics/APE1707S-12-HF.pdf"
- note removed: "DATASHEET PERFECT PENTRU A INTELEGE BUCK CONVERTOR https://pdf.datasheet.live/datasheets-1/advanced_power_electronics/APE1707S-12-HF.pdf"
- note removed: "Daca am nevoie de Vin la o tensiune mai mare(V) am nevoie de un alt chip(U2)"
- moved on the sheet: C1, C2, C3, C4, D1, L1, R1, R2, U2
